File: SMT/SeriesResonatorBlock_SMT.sch (KiCad schematic (older format))
At the start: 61 parts

Commit message: Completed Layout
Parts:
- removed UGY9, U_GY1, U_GY10, U_GY2, U_GY3, U_GY4, U_GY5, U_GY6, U_GY7, U_GY8: TL072, symbol TL072
- added U_GY1_2, U_GY3_4, U_GY5_6, U_GY7_8, U_GY9_10: TL072, Package_SO:SOIC-8_3.9x4.9mm_P1.27mm, symbol Amplifier_Operational:TL072
- C_GY1, C_GY10, C_GY2, C_GY3, C_GY4, C_GY5, C_GY6, C_GY7, C_GY8, C_GY9, C_PRE10, C_PRE2, C_PRE3, C_PRE4, C_PRE5, C_PRE6, C_PRE7, C_PRE8, C_PRE9, C_PREA1, C_PREB1: footprint (none) -> Capacitor_SMD:C_0805_2012Metric_Pad1.15x1.40mm_HandSolder; symbol C -> Device:C
- RV1, RV10, RV2, RV3, RV4, RV5, RV6, RV7, RV8, RV9: footprint (none) -> Bourn_PTA_Slider:PTA2043; symbol POT -> 1U_TenOctaveGraphicEQ_SMT-rescue:POT
- R_GYA1, R_GYA10, R_GYA2, R_GYA3, R_GYA4, R_GYA5, R_GYA6, R_GYA7, R_GYA8, R_GYA9, R_GYB1, R_GYB10, R_GYB2, R_GYB3, R_GYB4, R_GYB5, R_GYB6, R_GYB7, R_GYB8, R_GYB9: footprint (none) -> Resistor_SMD:R_0805_2012Metric_Pad1.15x1.40mm_HandSolder; symbol R -> Device:R
Connections:
- wire segments 182 -> 222
