File: THT/SeriesResonatorBlock_THT.sch (KiCad schematic (older format))
At the start: 61 parts

Commit message: Completed Layout
Parts:
- C_GY1, C_GY10, C_GY2, C_GY3, C_GY4, C_GY5, C_GY6, C_GY7, C_GY8, C_GY9, C_PRE10, C_PRE2, C_PRE3, C_PRE4, C_PRE5, C_PRE6, C_PRE7, C_PRE8, C_PRE9, C_PREA1, C_PREB1: symbol C -> Device:C
- RV1, RV10, RV2, RV3, RV4, RV5, RV6, RV7, RV8, RV9: symbol POT -> 1U_TenOctaveGraphicEQ_THT-rescue:POT
- R_GYA1, R_GYA10, R_GYA2, R_GYA3, R_GYA4, R_GYA5, R_GYA6, R_GYA7, R_GYA8, R_GYA9, R_GYB1, R_GYB10, R_GYB2, R_GYB3, R_GYB4, R_GYB5, R_GYB6, R_GYB7, R_GYB8, R_GYB9: symbol R -> Device:R
- UGY9, U_GY1, U_GY10, U_GY2, U_GY3, U_GY4, U_GY5, U_GY6, U_GY7, U_GY8: symbol TL072 -> 1U_TenOctaveGraphicEQ_THT-rescue:TL072
Changed lines of the file:
@@
-EESchema Schematic File Version 2
-LIBS:power
-LIBS:device
-LIBS:switches
-LIBS:relays
-LIBS:motors
-LIBS:transistors
-LIBS:conn
-LIBS:linear
-LIBS:regul
-LIBS:74xx
-LIBS:cmos4000
-LIBS:adc-dac
-LIBS:memory
-LIBS:xilinx
-LIBS:microcontrollers
-LIBS:dsp
-LIBS:microchip
-LIBS:analog_switches
-LIBS:motorola
-LIBS:texas
-LIBS:intel
-LIBS:audio
-LIBS:interface
-LIBS:digital-audio
-LIBS:philips
-LIBS:display
-LIBS:cypress
-LIBS:siliconi
-LIBS:opto
-LIBS:atmel
-LIBS:contrib
-LIBS:valves
-LIBS:_tc7662b
-LIBS:socket_custom
+EESchema Schematic File Version 4
 LIBS:1U_TenOctaveGraphicEQ_THT-cache
-EELAYER 25 0
+EELAYER 26 0
 EELAYER END
 $Descr A4 11693 8268
@@
 $EndDescr
 $Comp
-L TL072 U_GY1
+L 1U_TenOctaveGraphicEQ_THT-rescue:TL072 U_GY1
 U 1 1 5B7DC9E8
 P 3700 2550
@@
 $EndComp
 $Comp
-L TL072 U_GY2
+L 1U_TenOctaveGraphicEQ_THT-rescue:TL072 U_GY2
 U 1 1 5B7DC9EF
 P 4800 2550
@@
 	3600 2850 3600 2950
 $Comp
-L C C_GY1
+L Device:C C_GY1
 U 1 1 5B7DC9FA
 P 3200 2200
@@
 $EndComp
 $Comp
-L C C_PREB1
+L Device:C C_PREB1
 U 1 1 5B7DCA01
 P 3200 1700
@@
 $EndComp
 $Comp
-L R R_GYA1
+L Device:R R_GYA1
 U 1 1 5B7DCA08
 P 3650 1950
@@
 $EndComp
 $Comp
-L R R_GYB1
+L Device:R R_GYB1
 U 1 1 5B7DCA0F
 P 3200 3250
@@
 GND
 $Comp
-L POT RV1
+L 1U_TenOctaveGraphicEQ_THT-rescue:POT RV1
 U 1 1 5B7DCA25
 P 3650 1050
@@
 	4700 2850 4700 2950
 $Comp
-L C C_GY2
+L Device:C C_GY2
 U 1 1 5B7DCA32
 P 4300 2200
@@
 $EndComp
 $Comp
-L C C_PRE2
+L Device:C C_PRE2
 U 1 1 5B7DCA39
 P 4300 1700
@@
 $EndComp
 $Comp
-L R R_GYA2
+L Device:R R_GYA2
 U 1 1 5B7DCA40
 P 4750 1950
@@
 $EndComp
 $Comp
-L R R_GYB2
+L Device:R R_GYB2
 U 1 1 5B7DCA47
 P 4300 3250
@@
 GND
 $Comp
-L POT RV2
+L 1U_TenOctaveGraphicEQ_THT-rescue:POT RV2
 U 1 1 5B7DCA5D
 P 4750 1050
@@
 	4300 1050 4300 1550
 $Comp
-L TL072 U_GY3
+L 1U_TenOctaveGraphicEQ_THT-rescue:TL072 U_GY3
 U 1 1 5B7DD006
 P 5900 2550
@@
 $EndComp
 $Comp
-L TL072 U_GY4
+L 1U_TenOctaveGraphicEQ_THT-rescue:TL072 U_GY4
 U 1 1 5B7DD00C
 P 7000 2550
@@
 	5800 2850 5800 2950
 $Comp
-L C C_GY3
+L Device:C C_GY3
 U 1 1 5B7DD016
 P 5400 2200
@@
 $EndComp
 $Comp
-L C C_PRE3
+L Device:C C_PRE3
 U 1 1 5B7DD01C
 P 5400 1700
@@
 $EndComp
 $Comp
-L R R_GYA3
+L Device:R R_GYA3
 U 1 1 5B7DD022
 P 5850 1950
@@
 $EndComp
 $Comp
-L R R_GYB3
+L Device:R R_GYB3
 U 1 1 5B7DD028
 P 5400 3250
@@
 GND
 $Comp
-L POT RV3
+L 1U_TenOctaveGraphicEQ_THT-rescue:POT RV3
 U 1 1 5B7DD03D
 P 5850 1050
@@
 	6900 2850 6900 2950
 $Comp
-L C C_GY4
+L Device:C C_GY4
 U 1 1 5B7DD049
 P 6500 2200
@@
 $EndComp
 $Comp
-L C C_PRE4
+L Device:C C_PRE4
 U 1 1 5B7DD04F
 P 6500 1700
@@
 $EndComp
 $Comp
-L R R_GYA4
+L Device:R R_GYA4
 U 1 1 5B7DD055
 P 6950 1950
@@
 $EndComp
 $Comp
-L R R_GYB4
+L Device:R R_GYB4
 U 1 1 5B7DD05B
 P 6500 3250
@@
 GND
 $Comp
-L POT RV4
+L 1U_TenOctaveGraphicEQ_THT-rescue:POT RV4
 U 1 1 5B7DD070
 P 6950 1050
@@
 	6500 1050 6500 1550
 $Comp
-L TL072 U_GY5
+L 1U_TenOctaveGraphicEQ_THT-rescue:TL072 U_GY5
 U 1 1 5B7DD75B
 P 8100 2550
@@
 $EndComp
 $Comp
-L TL072 U_GY10
+L 1U_TenOctaveGraphicEQ_THT-rescue:TL072 U_GY10
 U 1 1 5B7DD761
 P 3700 5350
@@
 	8000 2850 8000 2950
 $Comp
-L C C_GY5
+L Device:C C_GY5
 U 1 1 5B7DD76B
 P 7600 2200
@@
 $EndComp
 $Comp
-L C C_PRE5
+L Device:C C_PRE5
 U 1 1 5B7DD771
 P 7600 1700
@@
 $EndComp
 $Comp
-L R R_GYA5
+L Device:R R_GYA5
 U 1 1 5B7DD777
 P 8050 1950
@@
 $EndComp
 $Comp
-L R R_GYB5
+L Device:R R_GYB5
 U 1 1 5B7DD77D
 P 7600 3250
@@
 GND
 $Comp
-L POT RV5
+L 1U_TenOctaveGraphicEQ_THT-rescue:POT RV5
 U 1 1 5B7DD795
 P 8050 1050
@@
 	3600 5650 3600 5750
 $Comp
-L C C_GY10
+L Device:C C_GY10
 U 1 1 5B7DD7A1
 P 3200 5000
@@
 $EndComp
 $Comp
-L C C_PRE10
+L Device:C C_PRE10
 U 1 1 5B7DD7A7
 P 3200 4500
@@
 $EndComp
 $Comp
-L R R_GYA10
+L Device:R R_GYA10
 U 1 1 5B7DD7AD
 P 3650 4750
@@
 $EndComp
 $Comp
-L R R_GYB10
+L Device:R R_GYB10
 U 1 1 5B7DD7B3
 P 3200 6050
@@
 GND
 $Comp
-L POT RV10
+L 1U_TenOctaveGraphicEQ_THT-rescue:POT RV10
 U 1 1 5B7DD7CB
 P 3650 4000
@@
 	3200 4000 3200 4350
 $Comp
-L TL072 UGY9
+L 1U_TenOctaveGraphicEQ_THT-rescue:TL072 UGY9
 U 1 1 5B7DD7D3
 P 4800 5350
@@
 $EndComp
 $Comp
-L TL072 U_GY8
+L 1U_TenOctaveGraphicEQ_THT-rescue:TL072 U_GY8
 U 1 1 5B7DD7D9
 P 5900 5350
@@
 	4700 5650 4700 5750
 $Comp
-L C C_GY9
+L Device:C C_GY9
 U 1 1 5B7DD7E3
 P 4300 5000
@@
 $EndComp
 $Comp
-L C C_PRE9
+L Device:C C_PRE9
 U 1 1 5B7DD7E9
 P 4300 4500
@@
 $EndComp
 $Comp
-L R R_GYA9
+L Device:R R_GYA9
 U 1 1 5B7DD7EF
 P 4750 4750
@@
 $EndComp
 $Comp
-L R R_GYB9
+L Device:R R_GYB9
 U 1 1 5B7DD7F5
 P 4300 6050
@@
 GND
 $Comp
-L POT RV9
+L 1U_TenOctaveGraphicEQ_THT-rescue:POT RV9
 U 1 1 5B7DD80D
 P 4750 4000
@@
 	5800 5650 5800 5750
 $Comp
-L C C_GY8
+L Device:C C_GY8
 U 1 1 5B7DD819
 P 5400 5000
@@
 $EndComp
 $Comp
-L C C_PRE8
+L Device:C C_PRE8
 U 1 1 5B7DD81F
 P 5400 4500
@@
 $EndComp
 $Comp
-L R R_GYA8
+L Device:R R_GYA8
 U 1 1 5B7DD825
 P 5850 4750
@@
 $EndComp
 $Comp
-L R R_GYB8
+L Device:R R_GYB8
 U 1 1 5B7DD82B
 P 5400 6050
@@
 GND
 $Comp
-L POT RV8
+L 1U_TenOctaveGraphicEQ_THT-rescue:POT RV8
 U 1 1 5B7DD843
 P 5850 4000
@@
 	5400 4000 5400 4350
 $Comp
-L TL072 U_GY7
+L 1U_TenOctaveGraphicEQ_THT-rescue:TL072 U_GY7
 U 1 1 5B7DDAAF
 P 7000 5350
@@
 $EndComp
 $Comp
-L TL072 U_GY6
+L 1U_TenOctaveGraphicEQ_THT-rescue:TL072 U_GY6
 U 1 1 5B7DDAB5
 P 8100 5350
@@
 	6900 5650 6900 5750
 $Comp
-L C C_GY7
+L Device:C C_GY7
 U 1 1 5B7DDABF
 P 6500 5000
@@
 $EndComp
 $Comp
-L C C_PRE7
+L Device:C C_PRE7
 U 1 1 5B7DDAC5
 P 6500 4500
@@
 $EndComp
 $Comp
-L R R_GYA7
+L Device:R R_GYA7
 U 1 1 5B7DDACB
 P 6950 4750
@@
 $EndComp
 $Comp
-L R R_GYB7
+L Device:R R_GYB7
 U 1 1 5B7DDAD1
 P 6500 6050
@@
 GND
 $Comp
-L POT RV7
+L 1U_TenOctaveGraphicEQ_THT-rescue:POT RV7
 U 1 1 5B7DDAE9
 P 6950 4000
@@
 	8000 5650 8000 5750
 $Comp
-L C C_GY6
+L Device:C C_GY6
 U 1 1 5B7DDAF5
 P 7600 5000
@@
 $EndComp
 $Comp
-L C C_PRE6
+L Device:C C_PRE6
 U 1 1 5B7DDAFB
 P 7600 4500
@@
 $EndComp
 $Comp
-L R R_GYA6
+L Device:R R_GYA6
 U 1 1 5B7DDB01
 P 8050 4750
@@
 $EndComp
 $Comp
-L R R_GYB6
+L Device:R R_GYB6
 U 1 1 5B7DDB07
 P 7600 6050
@@
 GND
 $Comp
-L POT RV6
+L 1U_TenOctaveGraphicEQ_THT-rescue:POT RV6
 U 1 1 5B7DDB1F
 P 8050 4000
@@
 EQ_IN
 $Comp
-L C C_PREA1
+L Device:C C_PREA1
 U 1 1 5B820882
 P 2800 1700
